File: hardware/FlipperZero_ARM_JTAG_Breakout_board/FlipperZero_ARM_JTAG_Breakout_board.kicad_pcb (KiCad board)
At the start: 2 copper layers, 64.5 x 36.8 mm, 24 parts, among them J1 ARM-JTAG, J10 nTRST_EN, J2 TC2050-IDC, J3 1.27mm, J4 TC2030-IDC, J5 SPI/ISP, J6 UART, J7 VTrefSel, J8 PWRSel, J9 RSTSel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

Commit message: added OSHWA Certification ID
Parts:
- LOGO1: value ~ -> BE000022
