File: hardware/FlipperZero_ARM_JTAG_Breakout_board/FlipperZero_ARM_JTAG_Breakout_board.kicad_sch (KiCad schematic)
At the start: 23 parts, among them J1 ARM-JTAG, J10 nTRST_EN, J2 TC2050-IDC, J3 1.27mm, J4 TC2030-IDC, J5 SPI/ISP, J6 UART, J7 VTrefSel, J8 PWRSel, J9 RSTSel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

Commit message: added OSHW footprint template
Parts:
- removed JP9: SolderJumper_2_Bridged, PCM_4ms_SolderJumper:JUMPER_SMD_1x2_tiny_shorted, symbol Jumper:SolderJumper_2_Bridged
- added JP9: TMS, PCM_4ms_SolderJumper:JUMPER_SMD_1x2_tiny, symbol Jumper:SolderJumper_2_Open
- added LOGO1: ~, OSHW:OSHW-Certification-Mark-Wide_4x25mm_SilkMask, symbol OSHW:OSHW_Certification_Mark_Stacked_Small
Connections:
- net CS: now also JP9.1 (A)
- net RSTSel: now also JP9.2 (B)
Changed lines of the file:
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@@
-	)
-	(junction
-		(at 114.3 104.14)
-		(diameter 0)
-		(color 0 0 0 0)
 	)
 	(junction
@@
 	(junction
 		(at 184.15 57.15)
+		(diameter 0)
+		(color 0 0 0 0)
+	)
+	(junction
+		(at 114.3 104.14)
 		(diameter 0)
 		(color 0 0 0 0)
@@
 	)
 	(symbol
-		(lib_id "Jumper:SolderJumper_2_Bridged")
-		(at 118.11 104.14 0)
-		(mirror x)
-		(unit 1)
-		(exclude_from_sim no)
-		(in_bom no)
-		(on_board yes)
-		(dnp no)
-		(property "Reference" "JP9"
-			(at 118.11 106.426 0)
-			(effects
-				(font
-					(size 1.27 1.27)
-				)
-			)
-		)
-		(property "Value" "SolderJumper_2_Bridged"
-			(at 118.11 107.95 0)
-			(effects
-				(font
-					(size 1.27 1.27)
-				)
-				(hide yes)
-			)
-		)
-		(property "Footprint" "PCM_4ms_SolderJumper:JUMPER_SMD_1x2_tiny_shorted"
-			(at 118.11 104.14 0)
-			(effects
-				(font
-					(size 1.27 1.27)
-				)
-				(hide yes)
-			)
-		)
-		(property "Datasheet" "~"
-			(at 118.11 104.14 0)
-			(effects
-				(font
-					(size 1.27 1.27)
-				)
-				(hide yes)
-			)
-		)
-		(property "Description" "Solder Jumper, 2-pole, closed/bridged"
-			(at 118.11 104.14 0)
-			(effects
-				(font
-					(size 1.27 1.27)
-				)
-				(hide yes)
-			)
-		)
-		(pin "1"
-		)
-		(pin "2"
-		)
-		(instances
-			(project "FlipperZero_ARM_JTAG_Breakout_board"
-				(path "/09bef04b-5b1b-4f9f-9366-e395bccbfbf5"
-					(reference "JP9")
-					(unit 1)
-				)
-			)
-		)
-	)
-	(symbol
 		(lib_id "Jumper:SolderJumper_2_Open")
 		(at 53.34 58.42 0)
@@
 	)
 	(symbol
+		(lib_id "OSHW:OSHW_Certification_Mark_Stacked_Small")
+		(at 34.29 189.23 0)
+		(unit 1)
+		(exclude_from_sim no)
+		(in_bom no)
+		(on_board no)
+		(dnp no)
+		(fields_autoplaced yes)
+		(property "Reference" "LOGO1"
+			(at 34.29 189.23 0)
+			(effects
+				(font
+					(size 1.27 1.27)
+				)
+				(hide yes)
+			)
+		)
+		(property "Value" "~"
+			(at 34.29 189.23 0)
+			(effects
+				(font
+					(size 1.27 1.27)
+				)
+				(hide yes)
+			)
+		)
+		(property "Footprint" "OSHW:OSHW-Certification-Mark-Wide_4x25mm_SilkMask"
+			(at 34.29 189.23 0)
+			(effects
+				(font
+					(size 1.27 1.27)
+				)
+				(hide yes)
+			)
+		)
+		(property "Datasheet" ""
+			(at 34.29 189.23 0)
+			(effects
+				(font
+					(size 1.27 1.27)
+				)
+				(hide yes)
+			)
+		)
+		(property "Description" "OSHW Certification Mark, Stacked"
+			(at 34.29 189.23 0)
+			(effects
+				(font
+					(size 1.27 1.27)
+				)
+				(hide yes)
+			)
+		)
+		(instances
+			(project ""
+				(path "/09bef04b-5b1b-4f9f-9366-e395bccbfbf5"
+					(reference "LOGO1")
+					(unit 1)
+				)
+			)
+		)
+	)
+	(symbol
 		(lib_id "Connector:Conn_01x04_Pin")
 		(at 74.93 101.6 0)
@@
 					(unit 1)
 				)
+			)
+		)
+	)
+	(symbol
+		(lib_id "Jumper:SolderJumper_2_Open")
+		(at 118.11 104.14 0)
+		(mirror x)
+		(unit 1)
+		(exclude_from_sim no)
+		(in_bom no)
+		(on_board yes)
+		(dnp no)
+		(property "Reference" "JP9"
+			(at 118.11 106.426 0)
+			(effects
+				(font
+					(size 1.27 1.27)
+				)
+			)
+		)
+		(property "Value" "TMS"
+			(at 118.11 101.854 0)
+			(effects
+				(font
+					(size 1.27 1.27)
+				)
+				(hide yes)
+			)
+		)
+		(property "Footprint" "PCM_4ms_SolderJumper:JUMPER_SMD_1x2_tiny"
+			(at 118.11 104.14 0)
+			(effects
+				(font
+					(size 1.27 1.27)
+				)
+				(hide yes)
+			)
+		)
+		(property "Datasheet" "~"
+			(at 118.11 104.14 0)
+			(effects
+				(font
+					(size 1.27 1.27)
+				)
+				(hide yes)
+			)
+		)
+		(property "Description" "Solder Jumper, 2-pole, open"
+			(at 118.11 104.14 0)
+			(effects
+				(font
+					(size 1.27 1.27)
+				)
+				(hide yes)
+			)
+		)
+		(pin "2"
+		)
+		(pin "1"
+		)
+		(instances
+			(project "FlipperZero_ARM_JTAG_Breakout_board"
+				(path "/09bef04b-5b1b-4f9f-9366-e395bccbfbf5"
+					(reference "JP9")
+					(unit 1)
+				)

Commit message: updated signal names for up-to-date terminology
Parts:
- A1: footprint Module:Flipper_Zero_Straight -> Module:Flipper_Zero_Angled
- LOGO1: footprint OSHW:OSHW-Certification-Mark-Wide_4x25mm_SilkMask -> OSHW:OSHW-Certification-Mark-Stacked_8x7mm_SilkMask
Connections:
- net MISO renamed SDI
- net MOSI renamed SDO
Changed lines of the file:
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@@
 		)
 	)
-	(label "MOSI"
+	(label "SDO"
 		(at 57.15 48.26 0)
 		(effects
@@
 		)
 	)
-	(label "MOSI"
+	(label "SDO"
 		(at 193.04 133.35 180)
 		(effects
@@
 		)
 	)
-	(label "MISO"
+	(label "SDI"
 		(at 157.48 130.81 0)
 		(effects
@@
 		)
 	)
-	(label "MISO"
+	(label "SDI"
 		(at 57.15 45.72 0)
 		(effects
@@
 		(exclude_from_sim no)
 		(in_bom no)
-		(on_board no)
+		(on_board yes)
 		(dnp no)
 		(fields_autoplaced yes)
@@
 			)
 		)
-		(property "Footprint" "OSHW:OSHW-Certification-Mark-Wide_4x25mm_SilkMask"
+		(property "Footprint" "OSHW:OSHW-Certification-Mark-Stacked_8x7mm_SilkMask"
 			(at 34.29 189.23 0)
 			(effects
@@
 			)
 		)
-		(property "Footprint" "Module:Flipper_Zero_Straight"
+		(property "Footprint" "Module:Flipper_Zero_Angled"
 			(at 82.55 81.534 0)
 			(effects

Commit message: updated footprint & ran DRU check
Parts:
- A1: footprint Module:Flipper_Zero_Angled -> Module:Flipper_Zero_Straight
Changed lines of the file:
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@@
 			)
 		)
-		(property "Footprint" "Module:Flipper_Zero_Angled"
+		(property "Footprint" "Module:Flipper_Zero_Straight"
 			(at 82.55 81.534 0)
 			(effects

Commit message: added OSHWA Certification ID
Parts:
- LOGO1: value ~ -> BE000022
Other:
- company: (none) -> Fred Corp.
- title: (none) -> FlipperZero JTAG/SWD/SPI breakout
Changed lines of the file:
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@@
 	(generator_version "9.0")
 	(paper "A4")
+	(title_block
+		(title "FlipperZero JTAG/SWD/SPI breakout")
+		(date "2025-11-14")
+		(rev "1")
+		(company "Fred Corp.")
+	)
 	(junction
 		(at 184.15 49.53)
@@
 	(symbol
 		(lib_id "OSHW:OSHW_Certification_Mark_Stacked_Small")
-		(at 34.29 189.23 0)
+		(at 280.67 184.15 0)
 		(unit 1)
 		(exclude_from_sim no)
@@
 		(fields_autoplaced yes)
 		(property "Reference" "LOGO1"
-			(at 34.29 189.23 0)
+			(at 280.67 184.15 0)
 			(effects
 				(font
@@
 			)
 		)
-		(property "Value" "~"
-			(at 34.29 189.23 0)
+		(property "Value" "BE000022"
+			(at 280.67 184.15 0)
 			(effects
 				(font
@@
 		)
 		(property "Footprint" "OSHW:OSHW-Certification-Mark-Stacked_8x7mm_SilkMask"
-			(at 34.29 189.23 0)
+			(at 280.67 184.15 0)
 			(effects
 				(font
@@
 		)
 		(property "Datasheet" ""
-			(at 34.29 189.23 0)
+			(at 280.67 184.15 0)
 			(effects
 				(font
@@
 		)
 		(property "Description" "OSHW Certification Mark, Stacked"
-			(at 34.29 189.23 0)
-			(effects
-				(font
+			(at 280.67 184.15 0)
+			(effects
+				(font
